Commit message: update adding camera and modify iiwa.launch.py

File: iiwa_description/urdf/iiwa.urdf.xacro (robot description, xacro)
@@ -5,4 +5,10 @@
     <color rgba="0.5 0.5 0.5 1.0"/>
   </material>
+  <material name="blu">
+    <color rgba="0 0 1 1"/>
+  </material>
+  <material name="red">
+    <color rgba="1 0 0 1"/>
+  </material>
   <link name="${prefix}iiwa_base" type="fixed"/>
   <joint name="${prefix}iiwa_root_joint" type="fixed">
@@ -170,4 +176,25 @@
   </link>
   <link name="${prefix}tool0"/>
+  <link name="${prefix}camera_link">
+    <visual>
+      <origin xyz="0 0 0" rpy="0 0 0"/>
+      <geometry>
+        <box size="0.03 0.03 0.03"/>
+      </geometry>
+      <material name="red"/>
+    </visual>
+    <collision>
+      <origin xyz="0 0 0" rpy="0 0 0"/>
+      <geometry>
+        <box size="0.03 0.03 0.03"/>
+      </geometry>
+    </collision>
+    <inertial>
+      <mass value="0.1" />
+      <origin xyz="0 0 0" rpy="0 0 0"/>
+      <inertia ixx="0.0001" ixy="0" ixz="0" iyy="0.0001" iyz="0" izz="0.0001" />
+    </inertial>
+  </link>
+  <link name="stereo_gazebo_right_camera_optical_frame"/>
   <joint name="${prefix}joint_a1" type="revolute">
       <origin rpy="0 0 0" xyz="0 0 0"/>
@@ -225,4 +252,33 @@
       <axis xyz="0 0 0"/>
   </joint>
+  <joint name="camera_joint" type="fixed">
+    <parent link="${prefix}tool0"/>
+    <child link="${prefix}camera_link"/>
+    <origin xyz="0 0 0.02" rpy="0 -1.5708 3.14"/>
+  </joint>
+  <joint name="camera_optical_joint" type="fixed">
+    <parent link="${prefix}camera_link"/>
+    <child link="stereo_gazebo_right_camera_optical_frame"/>
+    <origin xyz="0 0 0.02" rpy="-1.5708 0 -1.5708"/>
+  </joint>
+  <gazebo reference="${prefix}camera_link">
+    <sensor name="right_camera" type="camera">
+      <camera>
+        <horizontal_fov>1.047</horizontal_fov>
+          <clip>
+            <near>0.1</near>
+            <far>100</far>
+          </clip>
+          <image>
+              <width>640</width>
+              <height>480</height>
+          </image>
+      </camera>
+      <always_on>true</always_on>
+      <update_rate>10</update_rate>
+      <visualize>true</visualize>
+      <optical_frame_id>stereo_gazebo_right_camera_optical_frame</optical_frame_id>
+    </sensor>
+  </gazebo>
   </xacro:macro>
 </robot>
